Commit message: Included compatibility to run on real robot

File: ros2_ws/src/description/urdf/gripper/bio_gripper.gazebo.xacro (robot description, xacro)
@@ -30,4 +30,6 @@
   </xacro:macro>
   <xacro:macro name="bio_gazebo_grasp_fix" params="prefix:='' arm_name:='bio_gripper' palm_link:='link_base'">
+    <!-- Disabled by default: requires external libgazebo_grasp_fix.so -->
+    <!--
     <gazebo>
       <plugin name="gazebo_grasp_fix" filename="libgazebo_grasp_fix.so">
@@ -47,4 +49,5 @@
       </plugin>
     </gazebo>
+    -->
   </xacro:macro>
   <xacro:macro name="bio_gripper_gazebo" params="prefix">

File: ros2_ws/src/description/urdf/gripper_and_arm/arm_gripper_combined.urdf.xacro (robot description, xacro)
@@ -18,5 +18,5 @@
   <xacro:arg name="prefix"    default=""/>
   <xacro:arg name="hw_ns"     default="xarm"/>
-  <xacro:arg name="robot_ip"  default=""/>
+  <xacro:arg name="robot_ip"  default="192.168.1.212"/>
   <xacro:arg name="robot_sn"  default=""/>
   <xacro:arg name="limited"   default="false"/>
@@ -25,6 +25,8 @@
              default="uf_robot_hardware/UFRobotFakeSystemHardware"/>
   <xacro:arg name="use_gazebo" default="false"/>
+  <xacro:arg name="add_gripper_ros2_control" default="true"/>
   <!-- Property for conditional checks -->
   <xacro:property name="use_gazebo" value="$(arg use_gazebo)"/>
+  <xacro:property name="add_gripper_ros2_control_val" value="$(arg add_gripper_ros2_control)"/>
   <xacro:property name="is_ros2" value="true"/>
   <!-- ========== Include upstream xArm device macro ========== -->
@@ -64,9 +66,12 @@
     attach_rpy="0 0 0"
   />
-  <!-- ========== Add ros2_control interfaces for the gripper ========== -->
-  <xacro:bio_gripper_ros2_control
-    prefix="$(arg prefix)"
-    ros2_control_plugin="$(arg ros2_control_plugin)"
-  />
+  <!-- ========== Add ros2_control interfaces for the gripper (conditional) ========== -->
+  <!-- Skipped in real mode: the Dynamixel gripper is controlled independently -->
+  <xacro:if value="${add_gripper_ros2_control_val}">
+    <xacro:bio_gripper_ros2_control
+      prefix="$(arg prefix)"
+      ros2_control_plugin="$(arg ros2_control_plugin)"
+    />
+  </xacro:if>
   <!-- ========== Gazebo-specific Configuration ========== -->
   <!--
