Commit message: tcp calibration

File: ros2_ws/src/catalyst_description/urdf/gripper/bio_gripper.urdf.xacro (robot description, xacro)
@@ -18,5 +18,5 @@
       </inertial>
       <visual>
-        <origin xyz="0 0 0" rpy="0 0 0"/>
+        <origin rpy="1.57 0 1.57" xyz="0 0 0.039"/>
         <geometry>
           <mesh filename="file://$(find catalyst_description)/meshes/gripper/link_base.stl"/>
@@ -25,5 +25,5 @@
       </visual>
       <collision>
-        <origin xyz="0 0 0" rpy="0 0 0"/>
+        <origin rpy="1.57 0 1.57" xyz="0 0 0.039"/>
         <geometry>
           <mesh filename="file://$(find catalyst_description)/meshes/gripper/link_base.stl"/>
@@ -40,5 +40,5 @@
       </inertial>
       <visual>
-        <origin xyz="0 0 0" rpy="0 0 0"/>
+        <origin rpy="0 -1.57 3.14" xyz="0.0215 -0.025 0.013"/>
         <geometry>
           <mesh filename="file://$(find catalyst_description)/meshes/gripper/left_finger.stl"/>
@@ -47,5 +47,5 @@
       </visual>
       <collision>
-        <origin xyz="0 0 0" rpy="0 0 0"/>
+        <origin rpy="0 -1.57 3.14" xyz="0.0215 -0.025 0.013"/>
         <geometry>
           <mesh filename="file://$(find catalyst_description)/meshes/gripper/left_finger.stl"/>
@@ -70,5 +70,5 @@
       </inertial>
       <visual>
-        <origin xyz="0 0 0" rpy="0 0 0"/>
+        <origin rpy="0 -1.57 0" xyz="0.0215 0.025 0.013"/>
         <geometry>
           <mesh filename="file://$(find catalyst_description)/meshes/gripper/right_finger.stl"/>
@@ -77,5 +77,5 @@
       </visual>
       <collision>
-        <origin xyz="0 0 0" rpy="0 0 0"/>
+        <origin rpy="0 -1.57 0" xyz="0.0215 0.025 0.013"/>
         <geometry>
           <mesh filename="file://$(find catalyst_description)/meshes/gripper/right_finger.stl"/>
@@ -92,5 +92,5 @@
     <link name="${prefix}link_tcp" />
     <joint name="${prefix}joint_tcp" type="fixed">
-      <origin xyz="0.135 0 0.055" rpy="0 0 0" />
+      <origin xyz="0.1546 0 0.0563" rpy="0 0 0" />
       <parent link="${prefix}bio_gripper_base_link" />
       <child link="${prefix}link_tcp" />
