Commit message: pick_place

File: ros2_ws/src/catalyst_description/urdf/gripper/bio_gripper.ros2_control.xacro (robot description, xacro)
@@ -9,4 +9,5 @@
       <joint name="${prefix}right_finger_joint">
         <command_interface name="position">
+          <param name="initial_value">0.04</param>
         </command_interface>
         <command_interface name="velocity">
@@ -14,5 +15,7 @@
           <param name="max">3.14</param>
         </command_interface>
-        <state_interface name="position"/>
+        <state_interface name="position">
+          <param name="initial_value">0.04</param>
+        </state_interface>
         <state_interface name="velocity"/>
       </joint>
@@ -20,5 +23,7 @@
         <param name="mimic">${prefix}right_finger_joint</param>
         <param name="multiplier">-1</param>
-        <state_interface name="position"/>
+        <state_interface name="position">
+          <param name="initial_value">-0.04</param>
+        </state_interface>
         <state_interface name="velocity"/>
       </joint>

File: ros2_ws/src/catalyst_description/urdf/gripper_and_arm/arm_gripper_combined.urdf.xacro (robot description, xacro)
@@ -25,8 +25,13 @@
              default="uf_robot_hardware/UFRobotFakeSystemHardware"/>
   <xacro:arg name="use_gazebo" default="false"/>
+  <xacro:arg name="add_gripper" default="true"/>
   <xacro:arg name="add_gripper_ros2_control" default="true"/>
+  <xacro:arg name="add_ft_sensor" default="false"/>
+  <xacro:arg name="ft_sensor_ip" default="192.168.2.1"/>
   <!-- Property for conditional checks -->
   <xacro:property name="use_gazebo" value="$(arg use_gazebo)"/>
+  <xacro:property name="add_gripper_val" value="$(arg add_gripper)"/>
   <xacro:property name="add_gripper_ros2_control_val" value="$(arg add_gripper_ros2_control)"/>
+  <xacro:property name="add_ft_sensor_val" value="$(arg add_ft_sensor)"/>
   <!-- ========== Include upstream xArm device macro ========== -->
   <xacro:include filename="$(find xarm_description)/urdf/xarm_device_macro.xacro"/>
@@ -52,24 +57,73 @@
     add_bio_gripper="false"
   />
+  <!-- ========== F/T Sensor cylindrical link between flange and gripper ========== -->
+  <!--
+    Physical OnRobot F/T sensor body: 68mm diameter x 68mm height cylinder.
+    Sits between link_eef (flange) and the bio gripper.
+  -->
+  <link name="$(arg prefix)ft_sensor_link">
+    <visual>
+      <origin xyz="0 0 0.034" rpy="0 0 0"/>
+      <geometry>
+        <cylinder radius="0.034" length="0.068"/>
+      </geometry>
+      <material name="DarkGrey">
+        <color rgba="0.3 0.3 0.3 1.0"/>
+      </material>
+    </visual>
+    <collision>
+      <origin xyz="0 0 0.034" rpy="0 0 0"/>
+      <geometry>
+        <cylinder radius="0.034" length="0.068"/>
+      </geometry>
+    </collision>
+    <inertial>
+      <origin xyz="0 0 0.034" rpy="0 0 0"/>
+      <mass value="0.3"/>
+      <inertia ixx="0.0001" ixy="0" ixz="0" iyy="0.0001" iyz="0" izz="0.00005"/>
+    </inertial>
+  </link>
+  <joint name="$(arg prefix)ft_sensor_joint" type="fixed">
+    <parent link="$(arg prefix)link_eef"/>
+    <child link="$(arg prefix)ft_sensor_link"/>
+    <origin xyz="0 0 0" rpy="0 0 0"/>
+  </joint>
   <!-- ========== Attach our bio gripper to the arm ========== -->
   <!--
     The xarm6 kinematic chain ends at:
-      link6 -> (fixed joint_eef) -> link_eef
-    The bio_gripper_urdf macro uses attach_to / attach_xyz / attach_rpy
-    to create a fixed joint to the parent link.
+      link6 -> (fixed joint_eef) -> link_eef -> (fixed ft_sensor_joint) -> ft_sensor_link
+    The bio_gripper attaches to the top of the F/T sensor cylinder (offset 0.068m in Z).
   -->
-  <xacro:bio_gripper_urdf
-    prefix="$(arg prefix)"
-    attach_to="$(arg prefix)link_eef"
-    attach_xyz="0 0 0"
-    attach_rpy="0 0 0"
-  />
-  <!-- ========== Add ros2_control interfaces for the gripper (conditional) ========== -->
-  <!-- Skipped in real mode: the Dynamixel gripper is controlled independently -->
-  <xacro:if value="${add_gripper_ros2_control_val}">
-    <xacro:bio_gripper_ros2_control
+  <xacro:if value="${add_gripper_val}">
+    <xacro:bio_gripper_urdf
       prefix="$(arg prefix)"
-      ros2_control_plugin="$(arg ros2_control_plugin)"
+      attach_to="$(arg prefix)ft_sensor_link"
+      attach_xyz="0.039 0 0.107"
+      attach_rpy="0 -1.5708 0"
     />
+    <!-- ========== Add ros2_control interfaces for the gripper (conditional) ========== -->
+    <!-- Skipped in real mode: the Dynamixel gripper is controlled independently -->
+    <xacro:if value="${add_gripper_ros2_control_val}">
+      <xacro:bio_gripper_ros2_control
+        prefix="$(arg prefix)"
+        ros2_control_plugin="$(arg ros2_control_plugin)"
+      />
+    </xacro:if>
+  </xacro:if>
+  <!-- ========== OnRobot F/T sensor (real hardware only) ========== -->
+  <!--
+    Adds the net_ft_driver ros2_control sensor interface so the existing
+    controller_manager can load force_torque_sensor_broadcaster.
+    The sensor sits physically between link_eef and the gripper.
+  -->
+  <xacro:if value="${add_ft_sensor_val}">
+    <xacro:include filename="$(find net_ft_description)/urdf/net_ft_sensor.ros2_control.xacro"/>
+    <xacro:net_ft_sensor_ros2_control
+      name="NetFtHardwareInterface"
+      sensor_type="onrobot"
+      ip_address="$(arg ft_sensor_ip)"
+      rdt_sampling_rate="500"
+      internal_filter_rate="0"
+      use_hardware_biasing="true"/>
   </xacro:if>
   <!-- ========== Gazebo-specific Configuration ========== -->
@@ -88,11 +142,13 @@
     />
     <!-- Gripper Gazebo settings (collision, etc.) -->
-    <xacro:bio_gripper_gazebo prefix="$(arg prefix)"/>
-    <!-- Grasp fix plugin for realistic grasping -->
-    <xacro:bio_gazebo_grasp_fix
-      prefix="$(arg prefix)"
-      arm_name="bio_gripper"
-      palm_link="$(arg prefix)bio_gripper_base_link"
-    />
+    <xacro:if value="${add_gripper_val}">
+      <xacro:bio_gripper_gazebo prefix="$(arg prefix)"/>
+      <!-- Grasp fix plugin for realistic grasping -->
+      <xacro:bio_gazebo_grasp_fix
+        prefix="$(arg prefix)"
+        arm_name="bio_gripper"
+        palm_link="$(arg prefix)bio_gripper_base_link"
+      />
+    </xacro:if>
   </xacro:if>
 </robot>
